File: pcb/open-oswst.kicad_pcb (KiCad board)
At the start: 2 copper layers, 70 x 50 mm, 17 parts

Commit message: rev6? I lost count
Parts:
- moved AMP 4.00 mm to (123.6, 151.0)
- moved AMP_SPK 4.00 mm to (123.6, 138.0)
- moved J2 4.00 mm to (158.4, 145.4)
- moved J3 4.00 mm to (158.4, 122.6)
- moved MIC 4.00 mm to (148.0, 154.0)
- moved BAT 1.00 mm to (125.0, 117.0)
- moved CHNL 1.00 mm to (149.0, 117.0)
- moved PA 1.00 mm to (139.0, 117.0)
- moved PTT 1.00 mm to (170.0, 117.0)
- moved SW 1.00 mm to (132.0, 117.0)
- moved VOL 1.00 mm to (160.0, 117.0)
Other:
- board text added: "open-oswst e1d08f2"
- board text removed: "open-oswst 4d31d95"
Changed lines of the file:
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@@
   )
   (gr_rect (start 113 113) (end 183 163) (stroke (width 0.1) (type solid)) (fill none) (layer "Edge.Cuts"))
-  (gr_text "open-oswst  4d31d95"
+  (gr_text "open-oswst  e1d08f2"
     (at 148.0 161)
     (layer "F.SilkS")
@@
   (footprint "JST_PH_B2B"
     (layer "F.Cu")
-    (at 125 118)
+    (at 125 117)
     (fp_text reference "BAT" (at 0 -2.5) (layer "F.SilkS")
       (effects (font (size 1 1) (thickness 0.15)))
@@
   (footprint "JST_PH_B2B"
     (layer "F.Cu")
-    (at 132 118)
+    (at 132 117)
     (fp_text reference "SW" (at 0 -2.5) (layer "F.SilkS")
       (effects (font (size 1 1) (thickness 0.15)))
@@
   (footprint "JST_PH_B2B"
     (layer "F.Cu")
-    (at 139 118)
+    (at 139 117)
     (fp_text reference "PA" (at 0 -2.5) (layer "F.SilkS")
       (effects (font (size 1 1) (thickness 0.15)))
@@
   (footprint "JST_PH_B4B"
     (layer "F.Cu")
-    (at 149 118)
+    (at 149 117)
     (fp_text reference "CHNL" (at 0 -2.5) (layer "F.SilkS")
       (effects (font (size 1 1) (thickness 0.15)))
@@
   (footprint "JST_PH_B4B"
     (layer "F.Cu")
-    (at 160 118)
+    (at 160 117)
     (fp_text reference "VOL" (at 0 -2.5) (layer "F.SilkS")
       (effects (font (size 1 1) (thickness 0.15)))
@@
   (footprint "JST_PH_B2B"
     (layer "F.Cu")
-    (at 170 118)
+    (at 170 117)
     (fp_text reference "PTT" (at 0 -2.5) (layer "F.SilkS")
       (effects (font (size 1 1) (thickness 0.15)))
@@
   (footprint "PinHeader_1x18_P2.54mm"
     (layer "F.Cu")
-    (at 158.41 126.57)
+    (at 158.41 122.57)
     (fp_text reference "J3" (at 0 -2.5) (layer "F.SilkS")
       (effects (font (size 1 1) (thickness 0.15)))
@@
   (footprint "PinHeader_1x18_P2.54mm"
     (layer "F.Cu")
-    (at 158.41 149.43)
+    (at 158.41 145.43)
     (fp_text reference "J2" (at 0 -2.5) (layer "F.SilkS")
       (effects (font (size 1 1) (thickness 0.15)))
@@
   (footprint "PinHeader_1x5_P2.54mm"
     (layer "F.Cu")
-    (at 148.0 158)
+    (at 148.0 154)
     (fp_text reference "MIC" (at 0 -2.5) (layer "F.SilkS")
       (effects (font (size 1 1) (thickness 0.15)))
@@
   (footprint "PinHeader_1x7_P2.54mm"
     (layer "F.Cu")
-    (at 123.62 155 180)
+    (at 123.62 151 180)
     (fp_text reference "AMP" (at 0 -2.5) (layer "F.SilkS")
       (effects (font (size 1 1) (thickness 0.15)))
@@
   (footprint "PinHeader_1x2_P3.5mm"
     (layer "F.Cu")
-    (at 123.62 142.046 180)
+    (at 123.62 138.046 180)
     (fp_text reference "AMP_SPK" (at 0 -2.5) (layer "F.SilkS")
       (effects (font (size 1 1) (thickness 0.15)))

Commit message: rev6 pcb
Other:
- board text added: "open-oswst a2b3f21"
- board text removed: "open-oswst e1d08f2"
Changed lines of the file:
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@@
   )
   (gr_rect (start 113 113) (end 183 163) (stroke (width 0.1) (type solid)) (fill none) (layer "Edge.Cuts"))
-  (gr_text "open-oswst  e1d08f2"
+  (gr_text "open-oswst  a2b3f21"
     (at 148.0 161)
     (layer "F.SilkS")

Commit message: only room for 1 knob
Parts:
- removed CHNL: , JST_PH_B4B
Connections:
- J3 pad GPIO2: VOL_B -> (no net)
- J3 pad GPIO5: CHNL_SW -> (no net)
- J3 pad GPIO6: CHNL_B -> VOL_B
- J3 pad GPIO7: CHNL_A -> (no net)
Other:
- board text added: "open-oswst dbc0ed0"
- board text removed: "open-oswst a2b3f21"
Changed lines of the file:
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@@
   (net 2 "GND")
   (net 3 "VSW")
-  (net 4 "CHNL_A")
-  (net 5 "CHNL_B")
-  (net 6 "CHNL_SW")
-  (net 7 "VOL_A")
-  (net 8 "VOL_B")
-  (net 9 "VOL_SW")
-  (net 10 "PTT")
-  (net 11 "SPK-")
-  (net 12 "SPK+")
-  (net 13 "MIC_OUT")
-  (net 14 "LRC")
-  (net 15 "BCLK")
-  (net 16 "DIN")
-  (net 17 "Ve")
+  (net 4 "VOL_A")
+  (net 5 "VOL_B")
+  (net 6 "VOL_SW")
+  (net 7 "PTT")
+  (net 8 "SPK-")
+  (net 9 "SPK+")
+  (net 10 "MIC_OUT")
+  (net 11 "LRC")
+  (net 12 "BCLK")
+  (net 13 "DIN")
+  (net 14 "Ve")
   (net_class "Default" ""
     (clearance 0.2)
@@
   )
   (gr_rect (start 113 113) (end 183 163) (stroke (width 0.1) (type solid)) (fill none) (layer "Edge.Cuts"))
-  (gr_text "open-oswst  a2b3f21"
+  (gr_text "open-oswst  dbc0ed0"
     (at 148.0 161)
     (layer "F.SilkS")
@@
   (footprint "JST_PH_B4B"
     (layer "F.Cu")
-    (at 149 117)
-    (fp_text reference "CHNL" (at 0 -2.5) (layer "F.SilkS")
+    (at 160 117)
+    (fp_text reference "VOL" (at 0 -2.5) (layer "F.SilkS")
       (effects (font (size 1 1) (thickness 0.15)))
     )
@@
       (drill 0.8)
       (layers *.Cu *.Mask)
-      (net 4 "CHNL_A")
+      (net 4 "VOL_A")
     )
     (pad "B" thru_hole circle
@@
       (drill 0.8)
       (layers *.Cu *.Mask)
-      (net 5 "CHNL_B")
+      (net 5 "VOL_B")
     )
     (pad "SW" thru_hole circle
@@
       (drill 0.8)
       (layers *.Cu *.Mask)
-      (net 6 "CHNL_SW")
+      (net 6 "VOL_SW")
     )
     (pad "GND" thru_hole circle
@@
     )
   )
-  (footprint "JST_PH_B4B"
-    (layer "F.Cu")
-    (at 160 117)
-    (fp_text reference "VOL" (at 0 -2.5) (layer "F.SilkS")
-      (effects (font (size 1 1) (thickness 0.15)))
-    )
-    (pad "A" thru_hole circle
-      (at -3.0 0)
-      (size 1.5 1.5)
-      (drill 0.8)
-      (layers *.Cu *.Mask)
-      (net 7 "VOL_A")
-    )
-    (pad "B" thru_hole circle
-      (at -1.0 0)
-      (size 1.5 1.5)
-      (drill 0.8)
-      (layers *.Cu *.Mask)
-      (net 8 "VOL_B")
-    )
-    (pad "SW" thru_hole circle
-      (at 1.0 0)
-      (size 1.5 1.5)
-      (drill 0.8)
-      (layers *.Cu *.Mask)
-      (net 9 "VOL_SW")
-    )
-    (pad "GND" thru_hole circle
-      (at 3.0 0)
-      (size 1.5 1.5)
-      (drill 0.8)
-      (layers *.Cu *.Mask)
-      (net 2 "GND")
-    )
-  )
   (footprint "JST_PH_B2B"
     (layer "F.Cu")
@@
       (drill 0.8)
       (layers *.Cu *.Mask)
-      (net 10 "PTT")
+      (net 7 "PTT")
     )
     (pad "2" thru_hole circle
@@
       (drill 0.8)
       (layers *.Cu *.Mask)
-      (net 11 "SPK-")
+      (net 8 "SPK-")
     )
     (pad "+" thru_hole circle
@@
       (drill 0.8)
       (layers *.Cu *.Mask)
-      (net 12 "SPK+")
+      (net 9 "SPK+")
     )
   )
@@
       (drill 1.0)
       (layers *.Cu *.Mask)
-      (net 4 "CHNL_A")
     )
     (pad "GPIO6" thru_hole circle
@@
       (drill 1.0)
       (layers *.Cu *.Mask)
-      (net 5 "CHNL_B")
+      (net 5 "VOL_B")
     )
     (pad "GPIO5" thru_hole circle
@@
       (drill 1.0)
       (layers *.Cu *.Mask)
-      (net 6 "CHNL_SW")
     )
     (pad "GPIO4" thru_hole circle
@@
       (drill 1.0)
       (layers *.Cu *.Mask)
-      (net 13 "MIC_OUT")
+      (net 10 "MIC_OUT")
     )
     (pad "GPIO3" thru_hole circle
@@
       (drill 1.0)
       (layers *.Cu *.Mask)
-      (net 7 "VOL_A")
+      (net 4 "VOL_A")
     )
     (pad "GPIO2" thru_hole circle
@@
       (drill 1.0)
       (layers *.Cu *.Mask)
-      (net 8 "VOL_B")
     )
     (pad "GPIO1" thru_hole circle
@@
       (drill 1.0)
       (layers *.Cu *.Mask)
-      (net 9 "VOL_SW")
+      (net 6 "VOL_SW")
     )
     (pad "GPIO38" thru_hole circle
@@
       (drill 1.0)
       (layers *.Cu *.Mask)
-      (net 14 "LRC")
+      (net 11 "LRC")
     )
     (pad "GPIO47" thru_hole circle
@@
       (drill 1.0)
       (layers *.Cu *.Mask)
-      (net 15 "BCLK")
+      (net 12 "BCLK")
     )
     (pad "GPIO33" thru_hole circle
@@
       (drill 1.0)
       (layers *.Cu *.Mask)
-      (net 16 "DIN")
+      (net 13 "DIN")
     )
     (pad "GPIO34" thru_hole circle
@@
       (drill 1.0)
       (layers *.Cu *.Mask)
-      (net 10 "PTT")
+      (net 7 "PTT")
     )
     (pad "RST" thru_hole circle
@@
       (drill 1.0)
       (layers *.Cu *.Mask)
-      (net 17 "Ve")
+      (net 14 "Ve")
     )
     (pad "Ve_a" thru_hole circle
@@
       (drill 1.0)
       (layers *.Cu *.Mask)
-      (net 17 "Ve")
+      (net 14 "Ve")
     )
     (pad "5V" thru_hole circle
@@
       (drill 1.0)
       (layers *.Cu *.Mask)
-      (net 13 "MIC_OUT")
+      (net 10 "MIC_OUT")
     )
     (pad "GAIN" thru_hole circle
@@
       (drill 1.0)
       (layers *.Cu *.Mask)
-      (net 17 "Ve")
+      (net 14 "Ve")
     )
     (pad "GND" thru_hole circle
@@
       (drill 1.0)
       (layers *.Cu *.Mask)
-      (net 17 "Ve")
+      (net 14 "Ve")
     )
     (pad "GND" thru_hole circle
@@
       (drill 1.0)
       (layers *.Cu *.Mask)
-      (net 16 "DIN")
+      (net 13 "DIN")
     )
     (pad "BCLK" thru_hole circle
@@
       (drill 1.0)
       (layers *.Cu *.Mask)
-      (net 15 "BCLK")
+      (net 12 "BCLK")
     )
     (pad "LRC" thru_hole circle
@@
       (drill 1.0)
       (layers *.Cu *.Mask)
-      (net 14 "LRC")
+      (net 11 "LRC")
     )
   )
@@
       (drill 1.0)
       (layers *.Cu *.Mask)
-      (net 12 "SPK+")
+      (net 9 "SPK+")
     )
     (pad "-" thru_hole circle
@@
       (drill 1.0)
       (layers *.Cu *.Mask)
-      (net 11 "SPK-")
-    )
-  )
+      (net 8 "SPK-")
+    )
+  )

Commit message: pcb
Connections:
- J3 pad GPIO1: VOL_SW -> (no net)
- J3 pad GPIO45: (no net) -> VOL_SW
Other:
- board text added: "open-oswst 4468800"
- board text removed: "open-oswst dbc0ed0"
Changed lines of the file:
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@@
   )
   (gr_rect (start 113 113) (end 183 163) (stroke (width 0.1) (type solid)) (fill none) (layer "Edge.Cuts"))
-  (gr_text "open-oswst  dbc0ed0"
+  (gr_text "open-oswst  4468800"
     (at 148.0 161)
     (layer "F.SilkS")
@@
       (drill 1.0)
       (layers *.Cu *.Mask)
-      (net 6 "VOL_SW")
     )
     (pad "GPIO38" thru_hole circle
@@
       (drill 1.0)
       (layers *.Cu *.Mask)
+      (net 6 "VOL_SW")
     )
     (pad "GPIO46" thru_hole circle
